Commit message: Update camera joint position in parrot URDF

File: 41068_ignition_bringup/urdf_parrot/parrot.urdf.xacro (robot description, xacro)
@@ -82,5 +82,5 @@
   </link>
   <joint name="${prefix}camera_joint" type="fixed">
-    <origin xyz="0.25 0.0 0.25" rpy="0 0.785398 0"/> <!-- 0.5 0.0 0.9 -->
+    <origin xyz="0.0 0.0 -0.25" rpy="0 1.5708 0"/> <!-- 0.5 0.0 0.9 -->
     <parent link="${prefix}base_link"/>
     <child link="${prefix}camera_link"/>

Commit message: Fix camera joint origin position in URDF

File: 41068_ignition_bringup/urdf_parrot/parrot.urdf.xacro (robot description, xacro)
@@ -82,5 +82,5 @@
   </link>
   <joint name="${prefix}camera_joint" type="fixed">
-    <origin xyz="0.0 0.0 -0.25" rpy="0 1.5708 0"/> <!-- 0.5 0.0 0.9 -->
+    <origin xyz="0.0 0.0 0.0" rpy="0 1.5708 0"/> <!-- 0.5 0.0 0.9 -->
     <parent link="${prefix}base_link"/>
     <child link="${prefix}camera_link"/>
